Commit message: add posemonitor

File: RS-M90E7A.urdf (robot description, URDF)
Before this commit: robot RS-M90E7A, 13 links, 12 joints
Links:
- link base_link: mass 1.8420984607300377 -> 3.33
- link link1_1: mass 1.0 -> 5.310
- link link2_1: mass 1. -> 13.209
- link link3_1: mass 1. -> 5.306
- link link4_3_1: mass 1. -> 2.63
- link link5_1: mass 1. -> 2.63
- link link6_1: mass 1. -> 0.58
Joints:
- joint Revolute2: limit lower=-3.1415927 upper=3.1415927 effort=100000. velocity=1.0471976 -> lower=-6.2831854 upper=6.2831854 effort=100000. velocity=6.63225115758
- joint Revolute3: limit lower=-3.1415927 upper=3.1415927 effort=100000. velocity=1.0471976 -> lower=-6.2831854 upper=6.2831854 effort=100000. velocity=6.63225115758
- joint Revolute4: limit lower=-3.1415927 upper=3.1415927 effort=100000. velocity=1.0471976 -> lower=-6.2831854 upper=6.2831854 effort=100000. velocity=6.63225115758
- joint Revolute5: limit lower=-3.1415927 upper=3.1415927 effort=100000. velocity=1.0471976 -> lower=-4.04916386 upper=1.25663706 effort=100000. velocity=6.10865238198
- joint Revolute6: limit lower=-3.1415927 upper=3.1415927 effort=100000. velocity=1.0471976 -> lower=-6.2831854 upper=6.2831854 effort=100000. velocity=4.10152374219
- joint Revolute7: limit lower=-3.1415927 upper=3.1415927 effort=100000. velocity=1.0471976 -> lower=-6.2831854 upper=6.2831854 effort=100000. velocity=4.10152374219
